Commit message: world loaded

File: deepracer_description/models/xacro/deepracer/deepracer.xacro (robot description, xacro)
@@ -16,5 +16,5 @@
   <xacro:arg name="agent_name" default="agent" />
   <!-- Default: Use front facing camera and LiDAR sensor -->
-  <xacro:arg name="sensor_type" default="front_facing_camera_and_lidar" />
+  <xacro:arg name="sensor_type" default="front_facing_camera" />
   <xacro:arg name="shell" default="deepracer.STL" />
   <xacro:arg name="agent_bitmask" default="0x01" />

File: deepracer_description/models/xacro/urdf/deepracer_front_facing_camera_urdf.xacro (robot description, xacro)
@@ -23,7 +23,7 @@
         rpy="0 0 0" />
       <mass value="1.9068" />
-	    <inertia ixx="0.004151895" ixy="0"             ixz="0"
-	                               iyy="0.010379737"   iyz="0"
-	                                                   izz="0.010379737" />
+      <inertia ixx="0.004151895" ixy="0" ixz="0"
+        iyy="0.010379737" iyz="0"
+        izz="0.010379737" />
     </inertial>
   </link>
@@ -33,14 +33,17 @@
     <child link="chassis" />
   </joint>
-  <link
-    name="left_rear_wheel">
-    <inertial>
-      <origin
-        xyz="0 0 0"
-        rpy="0 1.5707 1.5707" />
-     <mass value="0.042222" />
-	   <inertia ixx="0.0000611771" ixy="0"            ixz="0"
-	                               iyy="0.0000611771" iyz="0"
-	                                                  izz="0.0000944606" />
+  <link name="left_rear_wheel">
+    <inertial>
+      <origin
+        xyz="0 0 0"
+        rpy="0 1.5707 1.5707" />
+      <mass value="0.042222" />
+      <inertia
+        ixx="0.0000611771"
+        ixy="0"
+        ixz="0"
+        iyy="0.0000611771"
+        iyz="0"
+        izz="0.0000944606" />
     </inertial>
     <visual>
@@ -61,6 +64,5 @@
     </collision>
   </link>
-  <joint
-    name="left_rear_wheel_joint"
+  <joint name="left_rear_wheel_joint"
     type="continuous">
     <origin
@@ -79,14 +81,13 @@
       velocity="100" />
   </joint>
-  <link
-    name="right_rear_wheel">
-    <inertial>
-      <origin
-        xyz="0 0 0"
-        rpy="0 1.5707 1.5707" />
-     <mass value="0.042222" />
-	   <inertia ixx="0.0000611771" ixy="0"            ixz="0"
-	                               iyy="0.0000611771" iyz="0"
-	                                                  izz="0.0000944606" />
+  <link name="right_rear_wheel">
+    <inertial>
+      <origin
+        xyz="0 0 0"
+        rpy="0 1.5707 1.5707" />
+      <mass value="0.042222" />
+      <inertia ixx="0.0000611771" ixy="0" ixz="0"
+        iyy="0.0000611771" iyz="0"
+        izz="0.0000944606" />
     </inertial>
     <visual>
@@ -107,6 +108,5 @@
     </collision>
   </link>
-  <joint
-    name="right_rear_wheel_joint"
+  <joint name="right_rear_wheel_joint"
     type="continuous">
     <origin
@@ -125,6 +125,5 @@
       velocity="100" />
   </joint>
-  <link
-    name="left_steering_hinge">
+  <link name="left_steering_hinge">
     <inertial>
       <origin
@@ -174,8 +173,8 @@
         xyz="0 0 0"
         rpy="0 1.5707 1.5707" />
-     <mass value="0.042222" />
-	   <inertia ixx="0.0000611771" ixy="0"            ixz="0"
-	                               iyy="0.0000611771" iyz="0"
-	                                                  izz="0.0000944606" />
+      <mass value="0.042222" />
+      <inertia ixx="0.0000611771" ixy="0" ixz="0"
+        iyy="0.0000611771" iyz="0"
+        izz="0.0000944606" />
     </inertial>
     <visual>
@@ -220,5 +219,5 @@
         xyz="0 0 0"
         rpy="0 0 0" />
-        <mass value="0.050" />
+      <mass value="0.050" />
       <inertia
         ixx="4E-06"
@@ -259,12 +258,12 @@
   <link
     name="right_front_wheel">
-      <inertial>
-      <origin
-        xyz="0 0 0"
-        rpy="0 1.5707 1.5707" />
-     <mass value="0.042222" />
-	   <inertia ixx="0.0000611771" ixy="0"            ixz="0"
-	                               iyy="0.0000611771" iyz="0"
-	                                                  izz="0.0000944606" />
+    <inertial>
+      <origin
+        xyz="0 0 0"
+        rpy="0 1.5707 1.5707" />
+      <mass value="0.042222" />
+      <inertia ixx="0.0000611771" ixy="0" ixz="0"
+        iyy="0.0000611771" iyz="0"
+        izz="0.0000944606" />
     </inertial>
     <visual>

Commit message: deepracer codes added

File: deepracer_description/models/xacro/deepracer/deepracer.xacro (robot description, xacro)
@@ -16,5 +16,5 @@
   <xacro:arg name="agent_name" default="agent" />
   <!-- Default: Use front facing camera and LiDAR sensor -->
-  <xacro:arg name="sensor_type" default="front_facing_camera" />
+  <xacro:arg name="sensor_type" default="front_facing_camera_and_lidar" />
   <xacro:arg name="shell" default="deepracer.STL" />
   <xacro:arg name="agent_bitmask" default="0x01" />

File: deepracer_description/models/xacro/urdf/deepracer_front_facing_camera_urdf.xacro (robot description, xacro)
@@ -23,7 +23,7 @@
         rpy="0 0 0" />
       <mass value="1.9068" />
-      <inertia ixx="0.004151895" ixy="0" ixz="0"
-        iyy="0.010379737" iyz="0"
-        izz="0.010379737" />
+	    <inertia ixx="0.004151895" ixy="0"             ixz="0"
+	                               iyy="0.010379737"   iyz="0"
+	                                                   izz="0.010379737" />
     </inertial>
   </link>
@@ -33,17 +33,14 @@
     <child link="chassis" />
   </joint>
-  <link name="left_rear_wheel">
-    <inertial>
-      <origin
-        xyz="0 0 0"
-        rpy="0 1.5707 1.5707" />
-      <mass value="0.042222" />
-      <inertia
-        ixx="0.0000611771"
-        ixy="0"
-        ixz="0"
-        iyy="0.0000611771"
-        iyz="0"
-        izz="0.0000944606" />
+  <link
+    name="left_rear_wheel">
+    <inertial>
+      <origin
+        xyz="0 0 0"
+        rpy="0 1.5707 1.5707" />
+     <mass value="0.042222" />
+	   <inertia ixx="0.0000611771" ixy="0"            ixz="0"
+	                               iyy="0.0000611771" iyz="0"
+	                                                  izz="0.0000944606" />
     </inertial>
     <visual>
@@ -64,5 +61,6 @@
     </collision>
   </link>
-  <joint name="left_rear_wheel_joint"
+  <joint
+    name="left_rear_wheel_joint"
     type="continuous">
     <origin
@@ -81,13 +79,14 @@
       velocity="100" />
   </joint>
-  <link name="right_rear_wheel">
-    <inertial>
-      <origin
-        xyz="0 0 0"
-        rpy="0 1.5707 1.5707" />
-      <mass value="0.042222" />
-      <inertia ixx="0.0000611771" ixy="0" ixz="0"
-        iyy="0.0000611771" iyz="0"
-        izz="0.0000944606" />
+  <link
+    name="right_rear_wheel">
+    <inertial>
+      <origin
+        xyz="0 0 0"
+        rpy="0 1.5707 1.5707" />
+     <mass value="0.042222" />
+	   <inertia ixx="0.0000611771" ixy="0"            ixz="0"
+	                               iyy="0.0000611771" iyz="0"
+	                                                  izz="0.0000944606" />
     </inertial>
     <visual>
@@ -108,5 +107,6 @@
     </collision>
   </link>
-  <joint name="right_rear_wheel_joint"
+  <joint
+    name="right_rear_wheel_joint"
     type="continuous">
     <origin
@@ -125,5 +125,6 @@
       velocity="100" />
   </joint>
-  <link name="left_steering_hinge">
+  <link
+    name="left_steering_hinge">
     <inertial>
       <origin
@@ -173,8 +174,8 @@
         xyz="0 0 0"
         rpy="0 1.5707 1.5707" />
-      <mass value="0.042222" />
-      <inertia ixx="0.0000611771" ixy="0" ixz="0"
-        iyy="0.0000611771" iyz="0"
-        izz="0.0000944606" />
+     <mass value="0.042222" />
+	   <inertia ixx="0.0000611771" ixy="0"            ixz="0"
+	                               iyy="0.0000611771" iyz="0"
+	                                                  izz="0.0000944606" />
     </inertial>
     <visual>
@@ -219,5 +220,5 @@
         xyz="0 0 0"
         rpy="0 0 0" />
-      <mass value="0.050" />
+        <mass value="0.050" />
       <inertia
         ixx="4E-06"
@@ -258,12 +259,12 @@
   <link
     name="right_front_wheel">
-    <inertial>
-      <origin
-        xyz="0 0 0"
-        rpy="0 1.5707 1.5707" />
-      <mass value="0.042222" />
-      <inertia ixx="0.0000611771" ixy="0" ixz="0"
-        iyy="0.0000611771" iyz="0"
-        izz="0.0000944606" />
+      <inertial>
+      <origin
+        xyz="0 0 0"
+        rpy="0 1.5707 1.5707" />
+     <mass value="0.042222" />
+	   <inertia ixx="0.0000611771" ixy="0"            ixz="0"
+	                               iyy="0.0000611771" iyz="0"
+	                                                  izz="0.0000944606" />
     </inertial>
     <visual>
